File: Hardware/SparkFun_Qwiic_ADXL313.brd (EAGLE design)
At the start: 25.4 x 25.4 mm, 57 parts, among them J2 QWIIC_RA, J4 QWIIC_RA, U1 ADXL313

Commit message: Axis label correction
-also updated xyz letters to buzzard text labels
Parts:
- added U$17, U$21: (no value), output:X0
- added U$26, U$29: (no value), output:Y0
- added U$31, U$32: (no value), output:Z0
Other:
- board text removed: "X"
- board text removed: "Y"
- board text removed: "Z"
Changed lines of the file:
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@@
 <drawing>
 <settings>
-<setting alwaysvectorfont="no"/>
+<setting alwaysvectorfont="yes"/>
 <setting keepoldvectorfont="yes"/>
 <setting verticaltext="up"/>
@@
 <wire x1="25.4" y1="25.4" x2="25.4" y2="0" width="0.2032" layer="20"/>
 <wire x1="25.4" y1="0" x2="0" y2="0" width="0.2032" layer="20"/>
-<wire x1="19.685" y1="16.9672" x2="22.352" y2="16.9672" width="0.254" layer="21"/>
-<wire x1="19.685" y1="16.9672" x2="20.066" y2="16.5862" width="0.254" layer="21"/>
-<wire x1="19.685" y1="16.9672" x2="20.066" y2="17.3482" width="0.254" layer="21"/>
-<wire x1="22.352" y1="19.6342" x2="22.352" y2="16.9672" width="0.254" layer="21"/>
-<wire x1="22.352" y1="19.6342" x2="21.971" y2="19.2532" width="0.254" layer="21"/>
-<wire x1="22.352" y1="19.6342" x2="22.733" y2="19.2532" width="0.254" layer="21"/>
-<circle x="21.209" y="18.1102" radius="0.127" width="0.254" layer="21"/>
-<text x="22.4536" y="20.2692" size="1.016" layer="21" font="vector" ratio="15" align="center">X</text>
-<text x="19.2278" y="17.018" size="1.016" layer="21" font="vector" ratio="15" align="center">Y</text>
-<text x="20.5486" y="19.2278" size="1.016" layer="21" font="vector" ratio="15" align="center">Z</text>
-<circle x="21.209" y="18.1102" radius="0.523634375" width="0.1778" layer="21"/>
-<wire x1="21.336" y1="15.4178" x2="24.003" y2="15.4178" width="0.254" layer="22"/>
-<wire x1="21.336" y1="15.4178" x2="21.717" y2="15.7988" width="0.254" layer="22"/>
-<wire x1="21.336" y1="15.4178" x2="21.717" y2="15.0368" width="0.254" layer="22"/>
-<wire x1="24.003" y1="18.0848" x2="24.003" y2="15.4178" width="0.254" layer="22"/>
-<wire x1="24.003" y1="18.0848" x2="24.384" y2="17.7038" width="0.254" layer="22"/>
-<wire x1="24.003" y1="18.0848" x2="23.622" y2="17.7038" width="0.254" layer="22"/>
-<text x="23.9268" y="18.7706" size="1.016" layer="22" font="vector" ratio="15" rot="MR180" align="center">X</text>
-<text x="20.7264" y="15.494" size="1.016" layer="22" font="vector" ratio="15" rot="MR0" align="center">Y</text>
-<text x="21.9456" y="17.6276" size="1.016" layer="22" font="vector" ratio="15" rot="MR0" align="center">Z</text>
-<circle x="22.86" y="16.5608" radius="0.523634375" width="0.1778" layer="22"/>
-<wire x1="23.1648" y1="16.891" x2="22.5298" y2="16.256" width="0.1778" layer="22"/>
-<wire x1="23.1648" y1="16.256" x2="22.5298" y2="16.891" width="0.1778" layer="22"/>
+<wire x1="21.5138" y1="17.6784" x2="21.5138" y2="20.3454" width="0.254" layer="21"/>
+<wire x1="21.5138" y1="17.6784" x2="21.8948" y2="18.0594" width="0.254" layer="21"/>
+<wire x1="21.5138" y1="17.6784" x2="21.1328" y2="18.0594" width="0.254" layer="21"/>
+<wire x1="18.8468" y1="20.3454" x2="21.5138" y2="20.3454" width="0.254" layer="21"/>
+<wire x1="18.8468" y1="20.3454" x2="19.2278" y2="19.9644" width="0.254" layer="21"/>
+<wire x1="18.8468" y1="20.3454" x2="19.2278" y2="20.7264" width="0.254" layer="21"/>
+<circle x="20.3708" y="19.2024" radius="0.127" width="0.254" layer="21"/>
+<circle x="20.3708" y="19.2024" radius="0.523634375" width="0.1778" layer="21"/>
+<wire x1="23.9522" y1="16.0274" x2="23.9522" y2="18.6944" width="0.254" layer="22"/>
+<wire x1="23.9522" y1="16.0274" x2="23.5712" y2="16.4084" width="0.254" layer="22"/>
+<wire x1="23.9522" y1="16.0274" x2="24.3332" y2="16.4084" width="0.254" layer="22"/>
+<wire x1="21.2852" y1="18.6944" x2="23.9522" y2="18.6944" width="0.254" layer="22"/>
+<wire x1="21.2852" y1="18.6944" x2="21.6662" y2="19.0754" width="0.254" layer="22"/>
+<wire x1="21.2852" y1="18.6944" x2="21.6662" y2="18.3134" width="0.254" layer="22"/>
+<circle x="22.8092" y="17.5514" radius="0.523634375" width="0.1778" layer="22"/>
+<wire x1="22.479" y1="17.8562" x2="23.114" y2="17.2212" width="0.1778" layer="22"/>
+<wire x1="23.114" y1="17.8562" x2="22.479" y2="17.2212" width="0.1778" layer="22"/>
 <text x="1.016" y="12.827" size="1.27" layer="16" font="vector" ratio="15" rot="MR90" align="center">v10</text>
 <dimension x1="2.54" y1="22.86" x2="22.86" y2="22.86" x3="12.7" y3="31.75" textsize="1.27" textratio="15" layer="47" unit="inch" visible="yes"/>
@@
 <element name="U$20" library="output" package="#SCLK#0" value="" x="13.9446" y="1.7018" smashed="yes" rot="MR90"/>
 <element name="U$12" library="output" package="#_ADR#0" value="" x="23.8506" y="8.0772" smashed="yes" rot="MR90"/>
+<element name="U$17" library="output" package="X0" value="" x="20.5486" y="18.6944" smashed="yes" rot="MR0"/>
+<element name="U$21" library="output" package="X0" value="" x="18.3388" y="20.3454" smashed="yes"/>
+<element name="U$26" library="output" package="Y0" value="" x="23.8506" y="15.3416" smashed="yes" rot="MR0"/>
+<element name="U$29" library="output" package="Y0" value="" x="21.59" y="17.1196" smashed="yes"/>
+<element name="U$31" library="output" package="Z0" value="" x="21.717" y="16.637" smashed="yes" rot="MR0"/>
+<element name="U$32" library="output" package="Z0" value="" x="19.431" y="18.4658" smashed="yes"/>
 </elements>
 <signals>
